Commit message: feat(urdf): Add 40cm mast link and remount OpenManipulator-X arm

File: src/custom_bot_description/urdf/robot.urdf.xacro (robot description, xacro)
@@ -10,10 +10,37 @@
   <!-- 3. Instantiate the OpenManipulator-X -->
   <xacro:open_manipulator_x prefix="omx_" />
-  <!-- 4. Attach the arm to the TurtleBot4 -->
-  <!-- We attach the base of the arm (omx_link1) to the TurtleBot4's top sensor plate -->
+  <!-- 4. Attach the arm to the TurtleBot4 via a mast -->
+  <link name="mast_link">
+    <visual>
+      <origin xyz="0 0 0.2" rpy="0 0 0"/>
+      <geometry>
+        <cylinder length="0.4" radius="0.02"/>
+      </geometry>
+    </visual>
+    <collision>
+      <origin xyz="0 0 0.2" rpy="0 0 0"/>
+      <geometry>
+        <cylinder length="0.4" radius="0.02"/>
+      </geometry>
+    </collision>
+    <inertial>
+      <mass value="0.2"/>
+      <inertia ixx="0.1" ixy="0" ixz="0" iyy="0.1" iyz="0" izz="0.1"/>
+    </inertial>
+  </link>
+  <joint name="mast_joint" type="fixed">
+    <parent link="tower_sensor_plate"/>
+    <child link="mast_link"/>
+    <!-- slightly offset backwards if needed, or just centered -->
+    <origin xyz="-0.03 0 0" rpy="0 0 0"/>
+  </joint>
+  <gazebo reference="mast_link">
+    <material>Gazebo/Black</material>
+  </gazebo>
+  <!-- We attach the base of the arm (omx_link1) to the top of the mast -->
   <joint name="arm_mount_joint" type="fixed">
-    <parent link="tower_sensor_plate"/>
+    <parent link="mast_link"/>
     <child link="omx_link1"/>
-    <origin xyz="0 0 0" rpy="0 0 0"/>
+    <origin xyz="0 0 0.4" rpy="0 0 0"/>
   </joint>
   <!-- Gazebo plugins for OpenManipulator-X might need to be explicitly included if we want ROS2 control -->
