Commit message: feat(manipulation): implement Phase 4 MoveIt2 and reasoning node manipulation extensions

File: src/custom_bot_description/urdf/robot.urdf.xacro (robot description, xacro)
@@ -20,3 +20,45 @@
   <xacro:include filename="$(find open_manipulator_description)/gazebo/open_manipulator_x.gazebo.xacro" />
   <xacro:open_manipulator_x_gazebo prefix="omx_" />
+  <!-- 5. ROS2 Control for the arm in Gazebo -->
+  <ros2_control name="open_manipulator_x_controller" type="system">
+    <hardware>
+      <plugin>gz_ros2_control/GazeboSimSystem</plugin>
+    </hardware>
+    <joint name="omx_joint1">
+      <command_interface name="position"/>
+      <command_interface name="velocity"/>
+      <state_interface name="position"/>
+      <state_interface name="velocity"/>
+    </joint>
+    <joint name="omx_joint2">
+      <command_interface name="position"/>
+      <command_interface name="velocity"/>
+      <state_interface name="position"/>
+      <state_interface name="velocity"/>
+    </joint>
+    <joint name="omx_joint3">
+      <command_interface name="position"/>
+      <command_interface name="velocity"/>
+      <state_interface name="position"/>
+      <state_interface name="velocity"/>
+    </joint>
+    <joint name="omx_joint4">
+      <command_interface name="position"/>
+      <command_interface name="velocity"/>
+      <state_interface name="position"/>
+      <state_interface name="velocity"/>
+    </joint>
+    <joint name="omx_gripper_left_joint">
+      <command_interface name="position"/>
+      <command_interface name="velocity"/>
+      <state_interface name="position"/>
+      <state_interface name="velocity"/>
+    </joint>
+    <joint name="omx_gripper_right_joint">
+      <command_interface name="position"/>
+      <command_interface name="velocity"/>
+      <state_interface name="position"/>
+      <state_interface name="velocity"/>
+    </joint>
+  </ros2_control>
 </robot>

Commit message: feat(grasping): isolate cylinder grasping and bypass Nav2 for direct test

File: src/custom_bot_description/urdf/robot.urdf.xacro (robot description, xacro)
@@ -15,5 +15,5 @@
     <parent link="tower_sensor_plate"/>
     <child link="omx_link1"/>
-    <origin xyz="0 0 0" rpy="0 0 0"/>
+    <origin xyz="0.12 0 0" rpy="0 0 0"/>
   </joint>
   <!-- Gazebo plugins for OpenManipulator-X might need to be explicitly included if we want ROS2 control -->
