Commit message: feat: setup headless gazebo and obstacle avoidance navigation

File: src/custom_bot_description/urdf/turtlebot4.urdf.xacro (robot description, xacro)
@@ -29,5 +29,5 @@
   <xacro:property name="camera_mount_x_offset"         value="${-11.8*cm2m}"/>
   <xacro:property name="camera_mount_y_offset"         value="${0*cm2m}"/>
-  <xacro:property name="camera_mount_z_offset"         value="${5.257*cm2m}"/>
+  <xacro:property name="camera_mount_z_offset"         value="${45.257*cm2m}"/>
   <xacro:property name="oakd_pro_x_offset"             value="${5.84*cm2m}"/>
   <xacro:property name="oakd_pro_y_offset"             value="${0*cm2m}"/>
